File: EDS_ALARM/EDS_ALARM.sch (KiCad schematic (older format))
At the start: 29 parts, among them J1 USB_B_Micro, J2 Conn_01x06_Male, J3 73412-0110, SW1 SW_Push, U1 EKMC1601111, U2 CMWX1ZZABZ-078, U3 LT1117-3.3, Y1 8.0MHz

Commit message: s
Parts:
- removed C14, C15: 18p, Capacitor_SMD:C_0805_2012Metric_Pad1.15x1.40mm_HandSolder, symbol Device:C
- removed HS1: HS-131, symbol HS-131:HS-131
- removed RV1: R_Variable, symbol Device:R_Variable
- removed Y1: 8.0MHz, Crystal:Crystal_HC49-U-3Pin_Vertical, symbol Device:Crystal
- added R2: R_Variable, symbol Device:R_Variable
- added U4: TGS2611-E00, Sensor:TGS2611-E00-PAK, symbol SMOKE:TGS2611-E00
- kmtg1603: footprint (none) -> buzzer:KMTG16031
Connections:
- net labels added: SMK_OUT
- wire segments 85 -> 69
- no-connect marks 32 -> 34
Other:
- moved on the sheet: J2, U1, kmtg1603

Commit message: Finishing schematic
Parts:
- removed R2: R_Variable, symbol Device:R_Variable
- added D1, D2: LED, LED_SMD:LED_0805_2012Metric, symbol Device:LED
- added RV1: 23BR1KLFTR, 23BR1KLFTR:23B_1, symbol 23BR1KLFTR:23BR1KLFTR
- SW1: footprint (none) -> Button_Switch_SMD:SW_SPST_PTS645
- U4: symbol SMOKE:TGS2611-E00 -> EDS_ALARM-rescue:TGS2611-E00-SMOKE
Connections:
- net labels added: ADC3, LED2
- net labels removed: SMK_OUT, SmokeSensor
- wire segments 69 -> 82
- no-connect marks 34 -> 33
Other:
- moved on the sheet: J2, U1, kmtg1603

Commit message: Finished layout
Parts:
- U4: footprint Sensor:TGS2611-E00-PAK -> TGS2611-E00:TGS2611C00
- kmtg1603: footprint buzzer:KMTG16031 -> KMTG1603-1:KMTG16031
Changed lines of the file:
@@
 NoConn ~ 2900 5850
 NoConn ~ 2900 5950
-Wire Wire Line
-	7450 3750 7750 3750
-$Comp
-L power:+5V #PWR0128
-U 1 1 5E460DD4
-P 7750 3750
-F 0 "#PWR0128" H 7750 3600 50  0001 C CNN
-F 1 "+5V" H 7765 3923 50  0000 C CNN
-F 2 "" H 7750 3750 50  0001 C CNN
-F 3 "" H 7750 3750 50  0001 C CNN
-	1    7750 3750
-	1    0    0    -1
-$EndComp
-$Comp
-L power:+5V #PWR0129
-U 1 1 5E463432
-P 6400 3700
-F 0 "#PWR0129" H 6400 3550 50  0001 C CNN
-F 1 "+5V" H 6415 3873 50  0000 C CNN
-F 2 "" H 6400 3700 50  0001 C CNN
-F 3 "" H 6400 3700 50  0001 C CNN
-	1    6400 3700
-	1    0    0    -1
-$EndComp
-$Comp
-L power:GND #PWR0130
-U 1 1 5E465C14
-P 6400 4000
-F 0 "#PWR0130" H 6400 3750 50  0001 C CNN
-F 1 "GND" H 6405 3827 50  0000 C CNN
-F 2 "" H 6400 4000 50  0001 C CNN
-F 3 "" H 6400 4000 50  0001 C CNN
-	1    6400 4000
-	1    0    0    -1
-$EndComp
-Text Label 8600 3950 0    50   ~ 0
-ADC3
 $Comp
 L Device:LED D1
@@
 Wire Wire Line
 	8400 3000 8500 3000
-Wire Wire Line
-	6450 3750 6400 3750
-Wire Wire Line
-	6400 3750 6400 3700
-Wire Wire Line
-	6400 4000 6400 3950
-Wire Wire Line
-	6400 3950 6450 3950
 Text Label 2750 4650 2    50   ~ 0
 LED2
 Wire Wire Line
 	2900 4650 2750 4650
-$Comp
-L EDS_ALARM-rescue:TGS2611-E00-SMOKE U4
-U 1 1 5E458258
-P 6950 3850
-F 0 "U4" H 6950 4217 50  0000 C CNN
-F 1 "TGS2611-E00" H 6950 4126 50  0000 C CNN
-F 2 "Sensor:TGS2611-E00-PAK" H 6950 3850 50  0001 L BNN
-F 3 "" H 6950 3850 50  0001 C CNN
-	1    6950 3850
-	1    0    0    -1
-$EndComp
 $Comp
 L power:+3.3V #PWR0108
@@
 F 0 "kmtg1603" H 7052 2079 50  0000 L CNN
 F 1 "Buzzer" H 7052 1988 50  0000 L CNN
-F 2 "buzzer:KMTG16031" V 6875 2150 50  0001 C CNN
+F 2 "KMTG1603-1:KMTG16031" V 6875 2150 50  0001 C CNN
 F 3 "~" V 6875 2150 50  0001 C CNN
 	1    6900 2050
@@
 	1    8400 2350
 	1    0    0    -1
+$EndComp
+Wire Wire Line
+	8600 3950 8500 3950
+Text Label 8600 3950 0    50   ~ 0
+ADC3
+Wire Wire Line
+	7700 3950 7450 3950
+Wire Wire Line
+	7600 4050 7700 4050
+Wire Wire Line
+	7600 4100 7600 4050
+$Comp
+L power:GND #PWR0131
+U 1 1 5E548ED4
+P 7600 4100
+F 0 "#PWR0131" H 7600 3850 50  0001 C CNN
+F 1 "GND" H 7605 3927 50  0000 C CNN
+F 2 "" H 7600 4100 50  0001 C CNN
+F 3 "" H 7600 4100 50  0001 C CNN
+	1    7600 4100
+	-1   0    0    -1
 $EndComp
 $Comp
@@
 $EndComp
 $Comp
-L power:GND #PWR0131
-U 1 1 5E548ED4
-P 7600 4100
-F 0 "#PWR0131" H 7600 3850 50  0001 C CNN
-F 1 "GND" H 7605 3927 50  0000 C CNN
-F 2 "" H 7600 4100 50  0001 C CNN
-F 3 "" H 7600 4100 50  0001 C CNN
-	1    7600 4100
-	-1   0    0    -1
-$EndComp
-Wire Wire Line
-	7600 4100 7600 4050
-Wire Wire Line
-	7600 4050 7700 4050
-Wire Wire Line
-	8600 3950 8500 3950
-Wire Wire Line
-	7700 3950 7450 3950
+L EDS_ALARM-rescue:TGS2611-E00-SMOKE U4
+U 1 1 5E458258
+P 6950 3850
+F 0 "U4" H 6950 4217 50  0000 C CNN
+F 1 "TGS2611-E00" H 6950 4126 50  0000 C CNN
+F 2 "TGS2611-E00:TGS2611C00" H 6950 3850 50  0001 L BNN
+F 3 "" H 6950 3850 50  0001 C CNN
+	1    6950 3850
+	1    0    0    -1
+$EndComp
+Wire Wire Line
+	6400 3950 6450 3950
+Wire Wire Line
+	6400 4000 6400 3950
+Wire Wire Line
+	6400 3750 6400 3700
+Wire Wire Line
+	6450 3750 6400 3750
+$Comp
+L power:GND #PWR0130
+U 1 1 5E465C14
+P 6400 4000
+F 0 "#PWR0130" H 6400 3750 50  0001 C CNN
+F 1 "GND" H 6405 3827 50  0000 C CNN
+F 2 "" H 6400 4000 50  0001 C CNN
+F 3 "" H 6400 4000 50  0001 C CNN
+	1    6400 4000
+	1    0    0    -1
+$EndComp
+$Comp
+L power:+5V #PWR0129
+U 1 1 5E463432
+P 6400 3700
+F 0 "#PWR0129" H 6400 3550 50  0001 C CNN
+F 1 "+5V" H 6415 3873 50  0000 C CNN
+F 2 "" H 6400 3700 50  0001 C CNN
+F 3 "" H 6400 3700 50  0001 C CNN
+	1    6400 3700
+	1    0    0    -1
+$EndComp
+$Comp
+L power:+5V #PWR0128
+U 1 1 5E460DD4
+P 7750 3750
+F 0 "#PWR0128" H 7750 3600 50  0001 C CNN
+F 1 "+5V" H 7765 3923 50  0000 C CNN
+F 2 "" H 7750 3750 50  0001 C CNN
+F 3 "" H 7750 3750 50  0001 C CNN
+	1    7750 3750
+	1    0    0    -1
+$EndComp
+Wire Wire Line
+	7450 3750 7750 3750
 $EndSCHEMATC

Commit message: s
Parts:
- removed J2: Conn_01x06_Male, Connector_PinHeader_2.54mm:PinHeader_1x06_P2.54mm_Vertical, symbol Connector:Conn_01x06_Male
- added D3: LED, LED_SMD:LED_0805_2012Metric, symbol Device:LED
- added J2: Conn_01x05_Male, Connector_PinSocket_2.54mm:PinSocket_1x05_P2.54mm_Vertical, symbol Connector:Conn_01x05_Male
- added J4: Conn_01x02_Male, Connector_PinSocket_2.54mm:PinSocket_1x02_P2.54mm_Vertical, symbol Connector:Conn_01x02_Male
- added R2: 680, Resistor_SMD:R_0805_2012Metric_Pad1.15x1.40mm_HandSolder, symbol Device:R
- added R3, R5: ??, Resistor_SMD:R_0805_2012Metric_Pad1.15x1.40mm_HandSolder, symbol Device:R
- added R4: 10k, Resistor_SMD:R_0805_2012Metric_Pad1.15x1.40mm_HandSolder, symbol Device:R
- added SW2: SW_Push, Button_Switch_SMD:SW_SPST_PTS645, symbol Switch:SW_Push
Connections:
- net +3V3: now also U2.47 (TCXO_OUT), J2.1 (Pin_1), R2.2, SW2.1; no longer D1.2 (A)
- net DAC1: now also R5.2
- net GND: now also D3.1 (K), J2.3 (Pin_3), R4.2
- net LED2: now also R3.2; no longer D2.2 (A)
- net NRST: now also J2.5 (Pin_5)
- net SWCLK: now also J2.2 (Pin_2)
- net SWDIO: now also J2.4 (Pin_4)
- net RX: now reaches U2.18 (PA10/USART1_RX)
- net RX: now also J4.2 (Pin_2)
- net TX: now reaches U2.19 (PA9/USART1_TX)
- net TX: now also J4.1 (Pin_1)
- net at U2.21 (PA5/ADC5/DAC2): now also R4.1, SW2.2
- net at U2.45 (PH1/OSC_OUT): now also U2.46 (PH0/OSC_IN)
- new net: D1.2 (A), R2.1
- new net: D2.2 (A), R3.1
- new net: D3.2 (A), R5.1
- no-connect marks 33 -> 26
Other:
- moved on the sheet: C12, SW1, kmtg1603

Commit message: s
Parts:
- U2: footprint RF_Module:CMWX1ZZABZ -> RF_Module:CMWX1ZZABZ_NEW
Changed lines of the file:
@@
 F 0 "U2" H 3800 3150 50  0000 C CNN
 F 1 "CMWX1ZZABZ-078" H 3800 3050 50  0000 C CNN
-F 2 "RF_Module:CMWX1ZZABZ" H 3800 5050 50  0001 C CNN
+F 2 "RF_Module:CMWX1ZZABZ_NEW" H 3800 5050 50  0001 C CNN
 F 3 "https://wireless.murata.com/RFM/data/type_abz.pdf" H 6250 3550 50  0001 C CNN
 	1    3800 5050

Commit message: s
Parts:
- J1: footprint Connector_USB:USB_Mini-B_Lumberg_2486_01_Horizontal -> Connector_USB:USB_Micro-B_Wuerth_629105150521
Changed lines of the file:
@@
 F 0 "J1" H 2707 2267 50  0000 C CNN
 F 1 "USB_B_Micro" H 2707 2176 50  0000 C CNN
-F 2 "Connector_USB:USB_Mini-B_Lumberg_2486_01_Horizontal" H 2800 1750 50  0001 C CNN
+F 2 "Connector_USB:USB_Micro-B_Wuerth_629105150521" H 2800 1750 50  0001 C CNN
 F 3 "~" H 2800 1750 50  0001 C CNN
 	1    2650 1800
